File: Board/Board.kicad_pcb (KiCad board)
At the start: 2 copper layers, 0 parts

Commit message: update board
Parts:
- added ?: LOGO, LOGO, F.Cu at (109.5, 127.5)
- added D1: GREEN_LED, LED_THT:LED_D3.0mm, F.Cu at (109.0, 136.8)
- added D2: RED_LED, LED_THT:LED_D3.0mm, F.Cu at (116.0, 136.8)
- added DR1: TB6612FNG, LGDXRobot2:TB6612FNG, F.Cu at (150.5, 60.0)
- added DR2: TB6612FNG, LGDXRobot2:TB6612FNG, F.Cu at (124.4, 60.1)
- added J1: XT30 Female, Connector_AMASS:AMASS_XT30U-F_1x02_P5.0mm_Vertical, F.Cu at (166.0, 68.5)
- added MJ1: ~, Connector_JST:JST_PH_B6B-PH-K_1x06_P2.00mm_Vertical, F.Cu at (166.5, 44.0)
- added MJ2: ~, Connector_JST:JST_PH_B6B-PH-K_1x06_P2.00mm_Vertical, F.Cu at (144.9, 43.6)
- added MJ3: ~, Connector_JST:JST_PH_B6B-PH-K_1x06_P2.00mm_Vertical, F.Cu at (128.9, 44.6)
- added MJ4: ~, Connector_JST:JST_PH_B6B-PH-K_1x06_P2.00mm_Vertical, F.Cu at (109.0, 44.0)
- added R1: 220R, Resistor_THT:R_Axial_DIN0207_L6.3mm_D2.5mm_P7.62mm_Horizontal, F.Cu at (109.6, 142.0)
- added R2: 4k7, Resistor_THT:R_Axial_DIN0207_L6.3mm_D2.5mm_P7.62mm_Horizontal, F.Cu at (132.0, 112.6)
- added R3: 4k7, Resistor_THT:R_Axial_DIN0207_L6.3mm_D2.5mm_P7.62mm_Horizontal, F.Cu at (138.0, 114.8)
- added RS1: ~, LGDXRobot2:Relay, F.Cu at (122.5, 130.5)
- added S1: INA226, LGDXRobot2:INA226, F.Cu at (126.2, 106.0)
- added S2: INA226, LGDXRobot2:INA226, F.Cu at (143.8, 106.0)
- added U1: BlackPill, LGDXRobot2:BlackPill, F.Cu at (134.2, 83.9)
Routing:
- net /GND23: track 0.00 -> 163.4 mm
- net /PA8_MJ2CH2: track 0.00 -> 139.2 mm
- net /5V98: track 0.00 -> 132.7 mm
- net /PA9_MJ2CH1: track 0.00 -> 117.9 mm
- net /PA0_MJ3CH1: track 0.00 -> 107.6 mm
- net /GND47: track 0.00 -> 105.8 mm
- net /PA1_MJ3CH2: track 0.00 -> 104.6 mm
- net /5V99: track 0.00 -> 96.8 mm
- net /PB6_MJ1CH1: track 0.00 -> 66.5 mm
- net /PB7_MJ1CH2: track 0.00 -> 65.2 mm
- net /PA6_MJ4CH2: track 0.00 -> 58.7 mm
- net /PA7_M41CH1: track 0.00 -> 50.5 mm
- net /PA15_RS1: track 0.00 -> 49.8 mm
- net GND: track 0.00 -> 49.3 mm
- net /PA10_D2: track 0.00 -> 46.6 mm
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- added copper zone on B.Cu, net /GND47
- added copper zone on F.Cu, net /GND47
Other:
- board outline added: 75 x 110 mm

Commit message: new design
Parts:
- added REF**: MountingHole_3.2mm_M3, MountingHole:MountingHole_3.2mm_M3, F.Cu at (167.5, 140.0)
- added REF**: MountingHole_3.2mm_M3, MountingHole:MountingHole_3.2mm_M3, F.Cu at (102.5, 140.0)
- added REF**: MountingHole_3.2mm_M3, MountingHole:MountingHole_3.2mm_M3, F.Cu at (102.5, 40.0)
- added REF**: MountingHole_3.2mm_M3, MountingHole:MountingHole_3.2mm_M3, F.Cu at (167.5, 40.0)
- moved MJ3 38.0 mm to (128.5, 43.0), turned to 180 degrees
- moved MJ2 37.4 mm to (166.2, 47.0), turned to -90 degrees
- moved MJ4 36.5 mm to (145.5, 43.0), turned to 0 degrees
- moved MJ1 36.0 mm to (109.0, 47.0), turned to -90 degrees
- moved DR2 26.1 mm to (150.5, 60.0)
- moved DR1 26.1 mm to (124.4, 60.0)
- moved J1 3.01 mm to (165.8, 71.5)
- renumbered MJ2 to MJ1, MJ3 to MJ2, MJ1 to MJ3
Connections:
- DR1 pad 15: /PA2_DR1PWMB -> /PA5_DR1PWMB
- DR1 pad 16: /PC15_DR1BIN2 -> /PB10_DR1BIN2
- DR1 pad 17: /PC14_DR1BIN1 -> /PB2_DR1BIN1
- DR1 pad 21: /PB4_DR1AIN1 -> /PB0_DR1AIN1
- DR1 pad 22: /PB5_DR1AIN1 -> /PA4_DR1AIN2
- DR1 pad 23: /PB3_DR1PWMA -> /PA3_DR1PWMA
- DR2 pad 15: /PA5_DR2PWMB -> /PA2_DR2PWMB
- DR2 pad 16: /PB10_DR2BIN2 -> /PC15_DR2BIN2
- DR2 pad 17: /PB2_DR2BIN1 -> /PC14_DR2BIN1
- DR2 pad 21: /PB0_DR2AIN1 -> /PB4_DR2AIN1
- DR2 pad 22: /PA4_DR2AIN2 -> /PB5_DR2AIN1
- DR2 pad 23: /PA3_DR2PWMA -> /PB3_DR2PWMA
- MJ1 pad 3: /PA8_MJ2CH2 -> /PA7_MJ1CH2
- MJ1 pad 4: /PA9_MJ2CH1 -> /PA6_MJ1CH1
- MJ2 pad 3: /PA1_MJ3CH2 -> /PB6_MJ2CH2
- MJ2 pad 4: /PA0_MJ3CH1 -> /PB7_MJ2CH1
- MJ3 pad 3: /PB7_MJ1CH2 -> /PA0_MJ3CH2
- MJ3 pad 4: /PB6_MJ1CH1 -> /PA1_MJ3CH1
- MJ4 pad 3: /PA6_MJ4CH2 -> /PA8_MJ4CH2
- MJ4 pad 4: /PA7_M41CH1 -> /PA9_MJ4CH1
- U1 pad 10: /PA0_MJ3CH1 -> /PA0_MJ3CH2
- U1 pad 11: /PA1_MJ3CH2 -> /PA1_MJ3CH1
- U1 pad 12: /PA2_DR1PWMB -> /PA2_DR2PWMB
- U1 pad 13: /PA3_DR2PWMA -> /PA3_DR1PWMA
- U1 pad 14: /PA4_DR2AIN2 -> /PA4_DR1AIN2
- U1 pad 15: /PA5_DR2PWMB -> /PA5_DR1PWMB
- U1 pad 16: /PA6_MJ4CH2 -> /PA6_MJ1CH1
- U1 pad 17: /PA7_M41CH1 -> /PA7_MJ1CH2
- U1 pad 18: /PB0_DR2AIN1 -> /PB0_DR1AIN1
- U1 pad 20: /PB2_DR2BIN1 -> /PB2_DR1BIN1
- U1 pad 21: /PB10_DR2BIN2 -> /PB10_DR1BIN2
- U1 pad 29: /PA8_MJ2CH2 -> /PA8_MJ4CH2
- U1 pad 3: /PC14_DR1BIN1 -> /PC14_DR2BIN1
- U1 pad 30: /PA9_MJ2CH1 -> /PA9_MJ4CH1
- U1 pad 39: /PB3_DR1PWMA -> /PB3_DR2PWMA
- U1 pad 4: /PC15_DR1BIN2 -> /PC15_DR2BIN2
- U1 pad 40: /PB4_DR1AIN1 -> /PB4_DR2AIN1
- U1 pad 41: /PB5_DR1AIN1 -> /PB5_DR2AIN1
- U1 pad 42: /PB6_MJ1CH1 -> /PB6_MJ2CH2
- U1 pad 43: /PB7_MJ1CH2 -> /PB7_MJ2CH1
Routing:
- net /PA8_MJ2CH2: track 139.2 -> 0.00 mm
- net /PA8_MJ4CH2: track 0.00 -> 133.3 mm
- net /PA9_MJ2CH1: track 117.9 -> 0.00 mm
- net /PA9_MJ4CH1: track 0.00 -> 112.6 mm
- net /PA0_MJ3CH1: track 107.6 -> 0.00 mm
- net /PA1_MJ3CH2: track 104.6 -> 0.00 mm
- net /PA0_MJ3CH2: track 0.00 -> 103.5 mm
- net /PA1_MJ3CH1: track 0.00 -> 94.3 mm
- net /PB6_MJ1CH1: track 66.5 -> 0.00 mm
- net /PB7_MJ1CH2: track 65.2 -> 0.00 mm
- net /PB6_MJ2CH2: track 0.00 -> 62.0 mm
- net /PA6_MJ4CH2: track 58.7 -> 0.00 mm
- net /PB7_MJ2CH1: track 0.00 -> 57.5 mm
- net /PA6_MJ1CH1: track 0.00 -> 52.5 mm
- net /PA7_M41CH1: track 50.5 -> 0.00 mm
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- removed copper zone on B.Cu, net /GND47
- removed copper zone on F.Cu, net /GND47

Commit message: update
Connections:
- net /PB5_DR2AIN1 renamed /PB5_DR2AIN2
Changed lines of the file:
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@@
 	(net 23 "Net-(MJ3-MV-)")
 	(net 24 "Net-(MJ4-MV-)")
-	(net 25 "/PB5_DR2AIN1")
+	(net 25 "/PB5_DR2AIN2")
 	(net 26 "/PB3_DR2PWMA")
 	(net 27 "/PA2_DR2PWMB")
@@
 			(layers "*.Cu" "*.Mask")
 			(remove_unused_layers no)
-			(net 25 "/PB5_DR2AIN1")
+			(net 25 "/PB5_DR2AIN2")
 			(pinfunction "AIN2")
 			(pintype "input")
@@
 			(layers "*.Cu" "*.Mask")
 			(remove_unused_layers no)
-			(net 25 "/PB5_DR2AIN1")
+			(net 25 "/PB5_DR2AIN2")
 			(pinfunction "PB5")
 			(pintype "bidirectional")

Commit message: board hole
Parts:
- removed the REF** at (167.5, 140.0)
- removed the REF** at (102.5, 140.0)
- removed the REF** at (102.5, 40.0)
- removed the REF** at (167.5, 40.0)
- added REF**: MountingHole_4.3mm_M4, MountingHole:MountingHole_4.3mm_M4, F.Cu at (167.5, 40.0)
- added REF**: MountingHole_4.3mm_M4, MountingHole:MountingHole_4.3mm_M4, F.Cu at (167.5, 140.0)
- added REF**: MountingHole_4.3mm_M4, MountingHole:MountingHole_4.3mm_M4, F.Cu at (102.5, 140.0)
- added REF**: MountingHole_4.3mm_M4, MountingHole:MountingHole_4.3mm_M4, F.Cu at (102.5, 40.0)

Commit message: update files
Parts:
- removed ?: LOGO, LOGO
- added G***: LOGO, LOGO, F.Cu at (109.0, 126.5)
Routing:
- added copper zone on B.Cu, net /GND47
- added copper zone on F.Cu, net /GND47
