File: Board/Board.kicad_pcb (KiCad board)
At the start: 2 copper layers, 75 x 110 mm, 21 parts, among them J1 XT30 Female, U1 BlackPill

Commit message: fix board design
Parts:
- moved G*** 1.50 mm to (109.0, 125.0)
Connections:
- U1 pad 23: unconnected-(U1-GND-Pad23) -> /GND23
- U1 pad 24: /GND23 -> unconnected-(U1-3V3-Pad24)
Routing:
- net /GND23: track 176.7 -> 177.6 mm
- net /PA8_MJ4CH2: track 133.3 -> 132.4 mm
- net /PA9_MJ4CH1: track 112.6 -> 112.0 mm
Changed lines of the file:
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@@
 	(net 52 "unconnected-(U1-3V3-Pad48)")
 	(net 53 "unconnected-(U1-PA11-Pad32)")
-	(net 54 "unconnected-(U1-GND-Pad23)")
+	(net 54 "unconnected-(U1-3V3-Pad24)")
 	(net 55 "unconnected-(U1-PB14-Pad27)")
 	(net 56 "unconnected-(U1-PA12-Pad33)")
@@
 			(layers "*.Cu" "*.Mask")
 			(remove_unused_layers no)
-			(net 54 "unconnected-(U1-GND-Pad23)")
+			(net 8 "/GND23")
 			(pinfunction "GND")
-			(pintype "power_out+no_connect")
+			(pintype "power_out")
 			(thermal_bridge_angle 45)
 		)
@@
 			(layers "*.Cu" "*.Mask")
 			(remove_unused_layers no)
-			(net 8 "/GND23")
+			(net 54 "unconnected-(U1-3V3-Pad24)")
 			(pinfunction "3V3")
-			(pintype "power_out")
+			(pintype "power_out+no_connect")
 			(thermal_bridge_angle 45)
 		)
@@
 	(footprint "LOGO"
 		(layer "F.Cu")
-		(at 109 126.5)
+		(at 109 125)
 		(property "Reference" "G***"
 			(at 0 0 0)
@@
 	)
 	(segment
+		(start 115.26 68.24)
+		(end 112.6 70.9)
+		(width 0.5)
+		(layer "B.Cu")
+		(net 8)
+	)
+	(segment
 		(start 168.75 53.5)
 		(end 167.25 55)
@@
 	)
 	(segment
-		(start 115.14 76.28)
-		(end 115.14 76.14)
+		(start 112.6 70.9)
+		(end 112.6 76.28)
 		(width 0.5)
 		(layer "B.Cu")
@@
 	)
 	(segment
-		(start 115.26 67.62)
-		(end 115.26 76.16)
-		(width 0.5)
-		(layer "B.Cu")
-		(net 8)
-	)
-	(segment
 		(start 120.5 40.5)
 		(end 141.5 40.5)
@@
 	)
 	(segment
-		(start 141.5 40.5)
-		(end 153.5 40.5)
+		(start 115.26 67.62)
+		(end 115.26 68.24)
 		(width 0.5)
 		(layer "B.Cu")
@@
 	)
 	(segment
-		(start 115.26 76.16)
-		(end 115.14 76.28)
+		(start 141.5 40.5)
+		(end 153.5 40.5)
 		(width 0.5)
 		(layer "B.Cu")
@@
 	)
 	(segment
+		(start 161.5 64)
+		(end 161.5 67.25)
+		(width 1.3)
+		(layer "B.Cu")
+		(net 15)
+	)
+	(segment
 		(start 165.75 71.5)
 		(end 165.75 71.25)
@@
 	)
 	(segment
-		(start 161 66.75)
-		(end 165.75 71.5)
+		(start 154.05 56.55)
+		(end 161.5 64)
 		(width 1.3)
 		(layer "B.Cu")
@@
 	)
 	(segment
-		(start 161 63.5)
-		(end 161 66.75)
+		(start 154.05 54.45)
+		(end 153 55.5)
 		(width 1.3)
 		(layer "B.Cu")
@@
 	)
 	(segment
-		(start 154.05 54.45)
-		(end 153 55.5)
+		(start 161.5 67.25)
+		(end 165.75 71.5)
 		(width 1.3)
 		(layer "B.Cu")
@@
 	)
 	(segment
-		(start 154.05 56.55)
-		(end 161 63.5)
-		(width 1.3)
-		(layer "B.Cu")
-		(net 15)
-	)
-	(segment
 		(start 138 76.28)
 		(end 138 72.7)
@@
 	)
 	(segment
-		(start 145.62 76.28)
-		(end 138.9 83)
+		(start 138.9 83)
+		(end 107 83)
 		(width 0.3)
 		(layer "F.Cu")
@@
 	)
 	(segment
-		(start 138.9 83)
-		(end 107 83)
+		(start 104 47.5)
+		(end 111 40.5)
 		(width 0.3)
 		(layer "F.Cu")
@@
 	)
 	(segment
-		(start 124.5 42)
-		(end 124.5 43)
+		(start 145.62 76.28)
+		(end 138.9 83)
 		(width 0.3)
 		(layer "F.Cu")
@@
 	)
 	(segment
-		(start 104 80)
-		(end 104 47)
+		(start 111 40.5)
+		(end 123 40.5)
 		(width 0.3)
 		(layer "F.Cu")
@@
 	)
 	(segment
-		(start 104 47)
-		(end 110.5 40.5)
+		(start 123 40.5)
+		(end 124.5 42)
 		(width 0.3)
 		(layer "F.Cu")
@@
 	)
 	(segment
-		(start 110.5 40.5)
-		(end 123 40.5)
+		(start 104 80)
+		(end 104 47.5)
 		(width 0.3)
 		(layer "F.Cu")
@@
 	)
 	(segment
-		(start 107 83)
-		(end 104 80)
+		(start 124.5 42)
+		(end 124.5 43)
 		(width 0.3)
 		(layer "F.Cu")
@@
 	)
 	(segment
-		(start 123 40.5)
-		(end 124.5 42)
+		(start 107 83)
+		(end 104 80)
 		(width 0.3)
 		(layer "F.Cu")
@@
 	)
 	(segment
-		(start 151 45.5)
-		(end 157 45.5)
+		(start 111 37.5)
+		(end 101 47.5)
 		(width 0.3)
 		(layer "F.Cu")
@@
 	)
 	(segment
-		(start 101 46)
-		(end 101 81)
+		(start 101 81)
+		(end 106 86)
+		(width 0.3)
+		(layer "F.Cu")
+		(net 35)
+	)
+	(segment
+		(start 151 45.5)
+		(end 157 45.5)
 		(width 0.3)
 		(layer "F.Cu")
@@
 	)
 	(segment
-		(start 109.5 37.5)
-		(end 101 46)
+		(start 101 47.5)
+		(end 101 81)
 		(width 0.3)
 		(layer "F.Cu")
@@
 	)
 	(segment
-		(start 157.5 45)
-		(end 157.5 42)
+		(start 153 37.5)
+		(end 111 37.5)
 		(width 0.3)
 		(layer "F.Cu")
@@
 	)
 	(segment
-		(start 101 81)
-		(end 106 86)
+		(start 149.5 44)
+		(end 151 45.5)
 		(width 0.3)
 		(layer "F.Cu")
@@
 	)
 	(segment
-		(start 157.5 42)
-		(end 153 37.5)
+		(start 114.72 86)
+		(end 120.22 91.5)
 		(width 0.3)
 		(layer "F.Cu")
@@
 	)
 	(segment
-		(start 149.5 44)
-		(end 151 45.5)
+		(start 157.5 45)
+		(end 157.5 42)
 		(width 0.3)
 		(layer "F.Cu")
@@
 	)
 	(segment
-		(start 153 37.5)
-		(end 109.5 37.5)
+		(start 157.5 42)
+		(end 153 37.5)
 		(width 0.3)
 		(layer "F.Cu")
@@
 	)
 	(segment
-		(start 114.72 86)
-		(end 120.22 91.5)
-		(width 0.3)
-		(layer "F.Cu")
-		(net 35)
-	)
-	(segment
-		(start 147.5 39)
-		(end 110 39)
+		(start 111 39)
+		(end 102.5 47.5)
 		(width 0.3)
 		(layer "F.Cu")
@@
 	)
 	(segment
-		(start 115.76 84.5)
-		(end 122.76 91.5)
+		(start 102.5 80.5)
+		(end 106.5 84.5)
 		(width 0.3)
 		(layer "F.Cu")
@@
 	)
 	(segment
-		(start 106.5 84.5)
-		(end 115.76 84.5)
+		(start 151.5 43)
+		(end 147.5 39)
 		(width 0.3)
 		(layer "F.Cu")
@@
 	)
 	(segment
-		(start 102.5 46.5)
+		(start 102.5 47.5)
 		(end 102.5 80.5)
 		(width 0.3)
@@
 	)
 	(segment
-		(start 110 39)
-		(end 102.5 46.5)
+		(start 115.76 84.5)
+		(end 122.76 91.5)
 		(width 0.3)
 		(layer "F.Cu")
@@
 	)
 	(segment
-		(start 102.5 80.5)
-		(end 106.5 84.5)
+		(start 147.5 39)
+		(end 111 39)
 		(width 0.3)
 		(layer "F.Cu")
@@
 	)
 	(segment
-		(start 151.5 43)
-		(end 147.5 39)
+		(start 106.5 84.5)
+		(end 115.76 84.5)
 		(width 0.3)
 		(layer "F.Cu")
@@
 		(net 45)
 	)
+	(segment
+		(start 115.14 76.28)
+		(end 115.14 76.14)
+		(width 0.5)
+		(layer "B.Cu")
+		(net 54)
+	)
+	(segment
+		(start 115.26 76.16)
+		(end 115.14 76.28)
+		(width 0.5)
+		(layer "B.Cu")
+		(net 54)
+	)
 	(zone

Commit message: board v2 pcb
Parts:
- removed D2: RED_LED, LED_THT:LED_D3.0mm
- removed G***: LOGO, LOGO
- removed S2: INA226, LGDXRobot2:INA226
- added C1: 0.1uF, Capacitor_THT:C_Disc_D5.0mm_W2.5mm_P2.50mm, F.Cu at (112.1, 128.2)
- added C2: 0.1uF, Capacitor_THT:C_Disc_D5.0mm_W2.5mm_P2.50mm, F.Cu at (112.0, 111.2)
- added C3: 0.1uF, Capacitor_THT:C_Disc_D5.0mm_W2.5mm_P2.50mm, F.Cu at (157.8, 110.5)
- added J2: PH2.0 2P, Connector_JST:JST_PH_B2B-PH-K_1x02_P2.00mm_Vertical, F.Cu at (117.1, 126.0)
- added J3: PH2.0 2P, Connector_JST:JST_PH_B2B-PH-K_1x02_P2.00mm_Vertical, F.Cu at (117.2, 109.0)
- added J4: PH2.0 2P, Connector_JST:JST_PH_B2B-PH-K_1x02_P2.00mm_Vertical, F.Cu at (155.5, 105.5)
- added R4: 68k, Resistor_THT:R_Axial_DIN0207_L6.3mm_D2.5mm_P7.62mm_Horizontal, F.Cu at (161.5, 105.5)
- added R5: 10k, Resistor_THT:R_Axial_DIN0207_L6.3mm_D2.5mm_P7.62mm_Horizontal, F.Cu at (109.5, 121.5)
- added R6: 10k, Resistor_THT:R_Axial_DIN0207_L6.3mm_D2.5mm_P7.62mm_Horizontal, F.Cu at (109.6, 105.0)
- added R7: 10k, Resistor_THT:R_Axial_DIN0207_L6.3mm_D2.5mm_P7.62mm_Horizontal, F.Cu at (151.5, 113.1)
- D1: value GREEN_LED -> RED_LED
- R2, R3: value 4k7 -> 68k
- S1: value INA226 -> ~; footprint LGDXRobot2:INA226 -> LGDXRobot2:ICM20948
- moved R2 24.4 mm to (117.1, 132.0), turned to 180 degrees
- moved R3 20.9 mm to (117.1, 115.0), turned to 180 degrees
- moved MJ1 13.8 mm to (122.5, 44.0), turned to 180 degrees
- moved S1 12.2 mm to (135.0, 114.5), turned to 0 degrees
- moved MJ3 10.5 mm to (139.0, 44.0)
- moved MJ2 7.67 mm to (159.0, 49.5), turned to 0 degrees
- moved J1 6.62 mm to (164.5, 65.0)
- moved DR2 6.16 mm to (144.9, 62.6)
- moved DR1 5.44 mm to (119.6, 62.5)
- moved U1 4.68 mm to (135.0, 88.5)
- moved D1 1.81 mm to (110.0, 138.3)
- moved R1 0.35 mm to (110.0, 142.0)
- moved RS1 0.05 mm to (122.5, 130.5)
Connections:
- D1 pad 2: /PB15_D1 -> /PB8_D1
- DR1 pad 15: /PA5_DR1PWMB -> /PA3_DR1PWMB
- DR1 pad 16: /PB10_DR1BIN2 -> /PB12_DR1BIN2
- DR1 pad 17: /PB2_DR1BIN1 -> /PB13_DR1BIN1
- DR1 pad 18: /GND23 -> /GND47
- DR1 pad 19: /PB1_DRxSTBY -> /PB2_DRxSTBY
- DR1 pad 21: /PB0_DR1AIN1 -> /PC15_DR1AIN1
- DR1 pad 22: /PA4_DR1AIN2 -> /PC14_DR1AIN2
- DR1 pad 23: /PA3_DR1PWMA -> /PA5_DR1PWMA
- DR2 pad 16: /PC15_DR2BIN2 -> /PC13_DR2BIN2
- DR2 pad 17: /PC14_DR2BIN1 -> /PA15_DR2BIN1
- DR2 pad 18: /GND23 -> /GND47
- DR2 pad 19: /PB1_DRxSTBY -> /PB2_DRxSTBY
- MJ1 pad 5: /GND23 -> /GND47
- MJ2 pad 5: /GND23 -> /GND47
- MJ3 pad 3: /PA0_MJ3CH2 -> /PA1_MJ3CH2
- MJ3 pad 4: /PA1_MJ3CH1 -> /PA0_MJ3CH1
- MJ3 pad 5: /GND23 -> /GND47
- MJ4 pad 5: /GND23 -> /GND47
- R2 pad 1: /5V99 -> Net-(J2-Pin_2)
- R2 pad 2: /PB9_SDA -> /PB1_BT1
- R3 pad 1: /5V99 -> Net-(J3-Pin_2)
- R3 pad 2: /PB8_SCL -> /PB0_BT2
- RS1 pad 3: /PA15_RS1 -> /PB9_RS1
- S1 pad 3: unconnected-(S1-~{Alert}-Pad3) -> /PB10_SCLK
- S1 pad 4: /PB9_SDA -> /PB15_SDA
- S1 pad 5: /PB8_SCL -> /PA10_NCS
- S1 pad 6: /5V99 -> /PB14_ADO
- S1 pad 7: /GND47 -> unconnected-(S1-INT-Pad7)
- S1 pad 8: /S1Vbus -> unconnected-(S1-FSY-Pad8)
- S1 pad 9: /S1Vbus -> unconnected-(S1-ACL-Pad9)
- U1 pad 10: /PA0_MJ3CH2 -> /PA0_MJ3CH1
- U1 pad 11: /PA1_MJ3CH1 -> /PA1_MJ3CH2
- U1 pad 13: /PA3_DR1PWMA -> /PA3_DR1PWMB
- U1 pad 14: /PA4_DR1AIN2 -> /PA4_ESTOP
- U1 pad 15: /PA5_DR1PWMB -> /PA5_DR1PWMA
- U1 pad 18: /PB0_DR1AIN1 -> /PB0_BT2
- U1 pad 19: /PB1_DRxSTBY -> /PB1_BT1
- U1 pad 2: unconnected-(U1-PC13-Pad2) -> /PC13_DR2BIN2
- U1 pad 20: /PB2_DR1BIN1 -> /PB2_DRxSTBY
- U1 pad 21: /PB10_DR1BIN2 -> /PB10_SCLK
- U1 pad 23: /GND23 -> unconnected-(U1-GND-Pad23)
- U1 pad 25: unconnected-(U1-PB12-Pad25) -> /PB12_DR1BIN2
- U1 pad 26: unconnected-(U1-PB13-Pad26) -> /PB13_DR1BIN1
- U1 pad 27: unconnected-(U1-PB14-Pad27) -> /PB14_ADO
- U1 pad 28: /PB15_D1 -> /PB15_SDA
- U1 pad 3: /PC14_DR2BIN1 -> /PC14_DR1AIN2
- U1 pad 31: /PA10_D2 -> /PA10_NCS
- U1 pad 38: /PA15_RS1 -> /PA15_DR2BIN1
- U1 pad 4: /PC15_DR2BIN2 -> /PC15_DR1AIN1
- U1 pad 45: /PB8_SCL -> /PB8_D1
- U1 pad 46: /PB9_SDA -> /PB9_RS1
- U1 pad 48: unconnected-(U1-3V3-Pad48) -> /3V348
Routing:
- net /GND47: track 105.8 -> 288.7 mm
- net /GND23: track 177.6 -> 0.00 mm
- net /PA0_MJ3CH1: track 0.00 -> 115.2 mm
- net /PA1_MJ3CH2: track 0.00 -> 113.7 mm
- net /PB8_D1: track 0.00 -> 111.1 mm
- net /PA4_ESTOP: track 0.00 -> 106.5 mm, vias 0 -> 1
- net /PA0_MJ3CH2: track 103.2 -> 0.00 mm
- net /PA1_MJ3CH1: track 94.3 -> 0.00 mm
- net /PB9_RS1: track 0.00 -> 91.3 mm
- net /PB1_BT1: track 0.00 -> 75.5 mm
- net /PB10_SCLK: track 0.00 -> 73.2 mm, vias 0 -> 1
- net /3V348: track 0.00 -> 67.0 mm
- net /PA15_DR2BIN1: track 0.00 -> 61.7 mm
- net /PB0_BT2: track 0.00 -> 57.3 mm
- net /PA15_RS1: track 49.8 -> 0.00 mm
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- removed copper zone on B.Cu, net /GND47
- removed copper zone on F.Cu, net /GND47
Other:
- board text added: "BT1"
- board text added: "BT2"
- board text added: "ESTOP"

Commit message: new board
Parts:
- added G***: LOGO, LOGO, F.Cu at (102.5, 118.5)
Routing:
- net /GND47: track 288.7 -> 294.8 mm
- added copper zone on B.Cu, net /GND47
- added copper zone on F.Cu, net /GND47

Commit message: update logo
Parts:
- moved G*** 0.50 mm to (102.5, 119.0)

Commit message: update logo
Parts:
- renumbered J2 to +J2, J3 to +J3, J4 to J4+
Changed lines of the file:
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@@
 		(descr "JST PH series connector, B2B-PH-K (http://www.jst-mfg.com/product/pdf/eng/ePH.pdf), generated with kicad-footprint-generator")
 		(tags "connector JST PH vertical")
-		(property "Reference" "J3"
+		(property "Reference" "+J3"
 			(at 1 -2.9 90)
 			(layer "F.SilkS")
@@
 		(descr "JST PH series connector, B2B-PH-K (http://www.jst-mfg.com/product/pdf/eng/ePH.pdf), generated with kicad-footprint-generator")
 		(tags "connector JST PH vertical")
-		(property "Reference" "J4"
+		(property "Reference" "J4+"
 			(at 1 -2.9 0)
 			(layer "F.SilkS")
@@
 		(descr "JST PH series connector, B2B-PH-K (http://www.jst-mfg.com/product/pdf/eng/ePH.pdf), generated with kicad-footprint-generator")
 		(tags "connector JST PH vertical")
-		(property "Reference" "J2"
+		(property "Reference" "+J2"
 			(at 1 -2.9 90)
 			(layer "F.SilkS")
@@
 		(at 122.5 130.54 -90)
 		(property "Reference" "RS1"
-			(at 0 2.5 90)
+			(at 10.96 0.25 90)
 			(layer "F.SilkS")
 			(effects
