File: Board/Board.kicad_sch (KiCad schematic)
At the start: 0 parts

Commit message: draw circuit
Parts:
- added D1: GREEN_LED, symbol Device:LED
- added D2: RED_LED, symbol Device:LED
- added DR1, DR2: TB6612FNG, Package_SO:SSOP-24_5.3x8.2mm_P0.65mm, symbol Driver_Motor:TB6612FNG
- added MJ1, MJ2, MJ3, MJ4: ~, symbol LGDXRobot2_Library:Motor_Socket
- added R1: 220R, symbol Device:R
- added R2, R3: 4k7, symbol Device:R
- added RS1: ~, symbol LGDXRobot2_Library:Relay_Socket
- added S1, S2: INA226, Package_SO:VSSOP-10_3x3mm_P0.5mm, symbol Sensor_Energy:INA226
- added U1: STM32F411CEU6, Package_DFN_QFN:QFN-48-1EP_7x7mm_P0.5mm_EP5.6x5.6mm, symbol MCU_ST_STM32F4:STM32F411CEUx
Connections:
- new net: D1.1 (K), D2.1 (K), R1.1
- new net: DR1.1 (AO1), DR1.2 (AO1), MJ1.1 (MV+)
- new net: DR1.10 (PGND2), DR1.9 (PGND2)
- new net: DR1.11 (BO1), DR1.12 (BO1), MJ2.1 (MV+)
- new net: DR1.5 (AO2), DR1.6 (AO2), MJ1.6 (MV-)
- new net: DR1.7 (BO2), DR1.8 (BO2), MJ2.6 (MV-)
- new net: DR2.11 (BO1), DR2.12 (BO1), MJ4.1 (MV+)
- new net: DR2.7 (BO2), DR2.8 (BO2), MJ4.6 (MV-)
- new net: DR2.1 (AO1), DR2.2 (AO1), MJ3.1 (MV+)
- new net: DR2.10 (PGND2), DR2.9 (PGND2)
- new net: DR2.5 (AO2), DR2.6 (AO2), MJ3.6 (MV-)
- new net: S2.8 (Vbus), S2.9 (Vin-)
- new net: S1.8 (Vbus), S1.9 (Vin-)
- new net: U1.23 (VSS), U1.35 (VSS), U1.47 (VSS), U1.49 (VSS)
- new net +12V: DR1.24 (VM1), DR2.24 (VM1)
- new net +5V: DR1.20 (VCC), DR2.20 (VCC), MJ1.5 (ENC_VCC), MJ2.5 (ENC_VCC), MJ3.5 (ENC_VCC), MJ4.5 (ENC_VCC), R2.1, R3.1, RS1.1 (VCC), S1.6 (VS), S2.6 (VS)
- new net GND: DR1.18 (GND), DR1.3 (PGND1), DR1.4 (PGND1), DR2.18 (GND), DR2.3 (PGND1), DR2.4 (PGND1), MJ1.2 (ENC_GND), MJ2.2 (ENC_GND), MJ3.2 (ENC_GND), MJ4.2 (ENC_GND), R1.2, RS1.2 (GND), S1.7 (GND), S2.7 (GND)
- new net PA0_MJ4CH2: MJ4.4 (ENC_CH2), U1.10 (PA0)
- new net PA10_DR2AIN2: DR2.22 (AIN2), U1.31 (PA10)
- new net PA15_DR2AIN1: DR2.21 (AIN1), U1.38 (PA15)
- new net PA1_MJ4CH1: MJ4.3 (ENC_CH1), U1.11 (PA1)
- new net PA2_DR2PWMB: DR2.15 (PWMB), U1.12 (PA2)
- new net PA3_DR1PWMA: DR1.23 (PWMA), U1.13 (PA3)
- new net PA4_DRxSTBY: DR1.19 (STBY), DR2.19 (STBY), U1.14 (PA4)
- new net PA5_DR1PWMB: DR1.15 (PWMB), U1.15 (PA5)
- new net PA6_MJ1CH1: MJ1.3 (ENC_CH1), U1.16 (PA6)
- new net PA7_MJ1CH2: MJ1.4 (ENC_CH2), U1.17 (PA7)
- new net PA8_MJ2CH2: MJ2.4 (ENC_CH2), U1.29 (PA8)
- new net PA9_MJ2CH1: MJ2.3 (ENC_CH1), U1.30 (PA9)
- new net PB10_RS1: RS1.3 (INPUT), U1.21 (PB10)
- new net PB12_DR1AIN2: DR1.22 (AIN2), U1.25 (PB12)
- new net PB13_DR1AIN1: DR1.21 (AIN1), U1.26 (PB13)
- new net PB14_DR1BIN1: DR1.17 (BIN1), U1.27 (PB14)
- new net PB15_DR1BIN2: DR1.16 (BIN2), U1.28 (PB15)
- new net PB1_D1: D1.2 (A), U1.19 (PB1)
- new net PB2_D2: D2.2 (A), U1.20 (PB2)
- new net PB3_DR2PWMA: DR2.23 (PWMA), U1.39 (PB3)
- new net PB4_DR2BIN1: DR2.17 (BIN1), U1.40 (PB4)
- new net PB5_DR2BIN2: DR2.16 (BIN2), U1.41 (PB5)
- new net PB6_MJ3CH1: MJ3.3 (ENC_CH1), U1.42 (PB6)
- new net PB7_MJ3CH2: MJ3.4 (ENC_CH2), U1.43 (PB7)
- new net PB8_SCL: R3.2, S1.5 (SCL), S2.5 (SCL), U1.45 (PB8)
- new net PB9_SDA: R2.2, S1.4 (SDA), S2.4 (SDA), U1.46 (PB9)
- no-connect marks 0 -> 34
Other:
- note added: "Microcontroller"
- note added: "Motor Drivers"
- note added: "Software E-STOP & Indicator"
- note added: "Voltage Sensors"

Commit message: footprint
Parts:
- removed U1: STM32F411CEU6, Package_DFN_QFN:QFN-48-1EP_7x7mm_P0.5mm_EP5.6x5.6mm, symbol MCU_ST_STM32F4:STM32F411CEUx
- added U1: BlackPill, LGDXRobot2:BlackPill, symbol LGDXRobot2_Library:BlackPill
- D1, D2: footprint (none) -> LED_THT:LED_D3.0mm
- DR1, DR2: footprint Package_SO:SSOP-24_5.3x8.2mm_P0.65mm -> LGDXRobot2:TB6612FNG
- MJ1, MJ2, MJ3, MJ4: footprint (none) -> Connector_JST:JST_PH_B6B-PH-K_1x06_P2.00mm_Vertical
- R1, R2, R3: footprint (none) -> Resistor_THT:R_Axial_DIN0207_L6.3mm_D2.5mm_P7.62mm_Horizontal
- RS1: footprint (none) -> Connector_PinHeader_2.54mm:PinHeader_1x03_P2.54mm_Vertical
- S1, S2: footprint Package_SO:VSSOP-10_3x3mm_P0.5mm -> LGDXRobot2:INA226
Connections:
- net GND: no longer DR1.18 (GND), DR2.18 (GND), MJ1.2 (ENC_GND), MJ2.2 (ENC_GND), MJ3.2 (ENC_GND), MJ4.2 (ENC_GND), R1.2, RS1.2 (GND), S1.7 (GND), S2.7 (GND)
- net PA0_MJ4CH2: now also U1.10 (PA0)
- net PA10_DR2AIN2: now also U1.31 (PA10)
- net PA15_DR2AIN1: now also U1.38 (PA15)
- net PA1_MJ4CH1: now also U1.11 (PA1)
- net PA2_DR2PWMB: now also U1.12 (PA2)
- net PA3_DR1PWMA: now also U1.13 (PA3)
- net PA4_DRxSTBY: now also U1.14 (PA4)
- net PA5_DR1PWMB: now also U1.15 (PA5)
- net PA6_MJ1CH1: now also U1.16 (PA6)
- net PA7_MJ1CH2: now also U1.17 (PA7)
- net PA8_MJ2CH2: now also U1.29 (PA8)
- net PA9_MJ2CH1: now also U1.30 (PA9)
- net PB10_RS1: now also U1.21 (PB10)
- net PB12_DR1AIN2: now also U1.25 (PB12)
- net PB13_DR1AIN1: now also U1.26 (PB13)
- net PB14_DR1BIN1: now also U1.27 (PB14)
- net PB15_DR1BIN2: now also U1.28 (PB15)
- net PB1_D1: now also U1.19 (PB1)
- net PB2_D2: now also U1.20 (PB2)
- net PB3_DR2PWMA: now also U1.39 (PB3)
- net PB4_DR2BIN1: now also U1.40 (PB4)
- net PB5_DR2BIN2: now also U1.41 (PB5)
- net PB6_MJ3CH1: now also U1.42 (PB6)
- net PB7_MJ3CH2: now also U1.43 (PB7)
- net PB8_SCL: now also U1.45 (PB8)
- net PB9_SDA: now also U1.46 (PB9)
- net +5V renamed 5V99
- net 5V99: now also U1.99 (5V); no longer RS1.1 (VCC)
- new net 5VD98: RS1.1 (VCC), U1.98 (5V)
- new net GND23: R1.2, RS1.2 (GND), U1.24 (3V3)
- new net GND47: DR1.18 (GND), DR2.18 (GND), MJ1.2 (ENC_GND), MJ2.2 (ENC_GND), MJ3.2 (ENC_GND), MJ4.2 (ENC_GND), S1.7 (GND), S2.7 (GND), U1.47 (GND)
- no-connect marks 34 -> 26

Commit message: net class
Connections:
- net DR1_A01: now reaches DR1.1 (AO1), DR1.2 (AO1), MJ1.1 (MV+)
- net DR1_B01: now reaches DR1.11 (BO1), DR1.12 (BO1), MJ2.1 (MV+)
- net DR1_A02: now reaches DR1.5 (AO2), DR1.6 (AO2), MJ1.6 (MV-)
- net DR1_B02: now reaches DR1.7 (BO2), DR1.8 (BO2), MJ2.6 (MV-)
- net DR2_B01: now reaches DR2.11 (BO1), DR2.12 (BO1), MJ4.1 (MV+)
- net DR2_B02: now reaches DR2.7 (BO2), DR2.8 (BO2), MJ4.6 (MV-)
- net DR2_A01: now reaches DR2.1 (AO1), DR2.2 (AO1), MJ3.1 (MV+)
- net DR2_A02: now reaches DR2.5 (AO2), DR2.6 (AO2), MJ3.6 (MV-)
- net S2Vbus: now reaches S2.8 (Vbus), S2.9 (Vin-)
- net S1Vbus: now reaches S1.8 (Vbus), S1.9 (Vin-)

Commit message: update board
Parts:
- added J1: XT30 Female, Connector_AMASS:AMASS_XT30U-F_1x02_P5.0mm_Vertical, symbol Connector:Conn_01x02_Socket
- RS1: footprint Connector_PinHeader_2.54mm:PinHeader_1x03_P2.54mm_Vertical -> LGDXRobot2:Relay
Connections:
- net +12V: now also J1.2 (Pin_2)
- net 5V99: now also RS1.1 (VCC); no longer DR1.20 (VCC), DR2.20 (VCC), MJ1.5 (ENC_VCC), MJ2.5 (ENC_VCC), MJ3.5 (ENC_VCC), MJ4.5 (ENC_VCC)
- net GND: now also J1.1 (Pin_1)
- net GND23: now also DR1.18 (GND), DR2.18 (GND), MJ1.5 (ENC_GND), MJ2.5 (ENC_GND), MJ3.5 (ENC_GND), MJ4.5 (ENC_GND); no longer R1.2, RS1.2 (GND)
- net GND47: now also R1.2, RS1.2 (GND); no longer DR1.18 (GND), DR2.18 (GND), MJ1.2 (ENC_GND), MJ2.2 (ENC_GND), MJ3.2 (ENC_GND), MJ4.2 (ENC_GND)
- net PA8_MJ2CH2: now also MJ2.3 (ENC_CH2); no longer MJ2.4 (ENC_CH2)
- net PA9_MJ2CH1: now also MJ2.4 (ENC_CH1); no longer MJ2.3 (ENC_CH1)
- net PB0_DR2AIN1: now reaches U1.18 (PB0)
- net PB0_DR2AIN1: now also DR2.21 (AIN1)
- net PC14_DR1BIN1: now reaches U1.3 (PC14)
- net PC14_DR1BIN1: now also DR1.17 (BIN1)
- net PC15_DR1BIN2: now reaches U1.4 (PC15)
- net PC15_DR1BIN2: now also DR1.16 (BIN2)
- net 5VD98 renamed 5V98
- net 5V98: now also DR1.20 (VCC), DR2.20 (VCC), MJ1.2 (ENC_VCC), MJ2.2 (ENC_VCC), MJ3.2 (ENC_VCC), MJ4.2 (ENC_VCC); no longer RS1.1 (VCC)
- net DR1_A01: no longer names the net of DR1.1 (AO1), DR1.2 (AO1)
- net DR1_A01: now also MJ1.6 (MV+); no longer MJ1.1 (MV+)
- net DR1_A02: no longer names the net of DR1.5 (AO2), DR1.6 (AO2)
- net DR1_A02: now also MJ1.1 (MV-); no longer MJ1.6 (MV-)
- net DR1_B01: no longer names the net of DR1.11 (BO1), DR1.12 (BO1)
- net DR1_B01: now also MJ2.6 (MV+); no longer MJ2.1 (MV+)
- net DR1_B02: no longer names the net of DR1.7 (BO2), DR1.8 (BO2)
- net DR1_B02: now also MJ2.1 (MV-); no longer MJ2.6 (MV-)
- net DR2_A01: no longer names the net of DR2.1 (AO1), DR2.2 (AO1)
- net DR2_A01: now also MJ3.6 (MV+); no longer MJ3.1 (MV+)
- net DR2_A02: no longer names the net of DR2.5 (AO2), DR2.6 (AO2)
- net DR2_A02: now also MJ3.1 (MV-); no longer MJ3.6 (MV-)
- net DR2_B01: no longer names the net of DR2.11 (BO1), DR2.12 (BO1)
- net DR2_B01: now also MJ4.6 (MV+); no longer MJ4.1 (MV+)
- net DR2_B02: no longer names the net of DR2.7 (BO2), DR2.8 (BO2)
- net DR2_B02: now also MJ4.1 (MV-); no longer MJ4.6 (MV-)
- net PA0_MJ4CH2 renamed PA0_MJ3CH1
- net PA0_MJ3CH1: now also MJ3.4 (ENC_CH1); no longer MJ4.4 (ENC_CH2)
- net PA10_DR2AIN2 renamed PA10_D2
- net PA10_D2: now also D2.2 (A); no longer DR2.22 (AIN2)
- net PA15_DR2AIN1 renamed PA15_RS1
- net PA15_RS1: now also RS1.3 (INPUT); no longer DR2.21 (AIN1)
- net PA1_MJ4CH1 renamed PA1_MJ3CH2
- net PA1_MJ3CH2: now also MJ3.3 (ENC_CH2); no longer MJ4.3 (ENC_CH1)
- net PA2_DR2PWMB renamed PA2_DR1PWMB
- net PA2_DR1PWMB: now also DR1.15 (PWMB); no longer DR2.15 (PWMB)
- net PA3_DR1PWMA renamed PA3_DR2PWMA
- net PA3_DR2PWMA: now also DR2.23 (PWMA); no longer DR1.23 (PWMA)
- net PA4_DRxSTBY renamed PB1_DRxSTBY
- net PB1_DRxSTBY: now also U1.19 (PB1); no longer U1.14 (PA4)
- net PA5_DR1PWMB renamed PA5_DR2PWMB
- net PA5_DR2PWMB: now also DR2.15 (PWMB); no longer DR1.15 (PWMB)
- net PA6_MJ1CH1 renamed PA6_MJ4CH2
- net PA6_MJ4CH2: now also MJ4.3 (ENC_CH2); no longer MJ1.3 (ENC_CH1)
- net PA7_MJ1CH2 renamed PA7_M41CH1
- net PA7_M41CH1: now also MJ4.4 (ENC_CH1); no longer MJ1.4 (ENC_CH2)
- net PB10_RS1 renamed PB10_DR2BIN2
- net PB10_DR2BIN2: now also DR2.16 (BIN2); no longer RS1.3 (INPUT)
- net PB12_DR1AIN2: no longer names the net of U1.25 (PB12)
- net PB12_DR1AIN2: no longer DR1.22 (AIN2)
- net PB13_DR1AIN1: no longer names the net of U1.26 (PB13)
- net PB13_DR1AIN1: no longer DR1.21 (AIN1)
- net PB14_DR1BIN1: no longer names the net of U1.27 (PB14)
- net PB14_DR1BIN1: no longer DR1.17 (BIN1)
- net PB15_DR1BIN2 renamed PB15_D1
- net PB15_D1: now also D1.2 (A); no longer DR1.16 (BIN2)
- removed net PB1_D1: D1.2 (A), U1.19 (PB1)
- net PB2_D2 renamed PB2_DR2BIN1
- net PB2_DR2BIN1: now also DR2.17 (BIN1); no longer D2.2 (A)
- net PB3_DR2PWMA renamed PB3_DR1PWMA
- net PB3_DR1PWMA: now also DR1.23 (PWMA); no longer DR2.23 (PWMA)
- net PB4_DR2BIN1 renamed PB4_DR1AIN1
- net PB4_DR1AIN1: now also DR1.21 (AIN1); no longer DR2.17 (BIN1)
- net PB5_DR2BIN2 renamed PB5_DR1AIN1
- net PB5_DR1AIN1: now also DR1.22 (AIN2); no longer DR2.16 (BIN2)
- net PB6_MJ3CH1 renamed PB6_MJ1CH1
- net PB6_MJ1CH1: now also MJ1.4 (ENC_CH1); no longer MJ3.3 (ENC_CH1)
- net PB7_MJ3CH2 renamed PB7_MJ1CH2
- net PB7_MJ1CH2: now also MJ1.3 (ENC_CH2); no longer MJ3.4 (ENC_CH2)
- new net PA4_DR2AIN2: DR2.22 (AIN2), U1.14 (PA4)
Other:
- moved on the sheet: MJ1, MJ2, MJ3, MJ4

Commit message: new design
Parts:
- renumbered MJ2 to MJ1, MJ3 to MJ2, MJ1 to MJ3
Connections:
- net PA0_MJ3CH1 renamed PA0_MJ3CH2
- net PA0_MJ3CH2: now also MJ3.3 (ENC_CH2); no longer MJ2.4 (ENC_CH1)
- net PA1_MJ3CH2 renamed PA1_MJ3CH1
- net PA1_MJ3CH1: now also MJ3.4 (ENC_CH1); no longer MJ2.3 (ENC_CH2)
- net PA2_DR1PWMB renamed PA2_DR2PWMB
- net PA2_DR2PWMB: now also DR2.15 (PWMB); no longer DR1.15 (PWMB)
- net PA3_DR2PWMA renamed PA3_DR1PWMA
- net PA3_DR1PWMA: now also DR1.23 (PWMA); no longer DR2.23 (PWMA)
- net PA4_DR2AIN2 renamed PA4_DR1AIN2
- net PA4_DR1AIN2: now also DR1.22 (AIN2); no longer DR2.22 (AIN2)
- net PA5_DR2PWMB renamed PA5_DR1PWMB
- net PA5_DR1PWMB: now also DR1.15 (PWMB); no longer DR2.15 (PWMB)
- net PA6_MJ4CH2 renamed PA6_MJ1CH1
- net PA6_MJ1CH1: now also MJ1.4 (ENC_CH1); no longer MJ4.3 (ENC_CH2)
- net PA7_M41CH1 renamed PA7_MJ1CH2
- net PA7_MJ1CH2: now also MJ1.3 (ENC_CH2); no longer MJ4.4 (ENC_CH1)
- net PA8_MJ2CH2 renamed PA8_MJ4CH2
- net PA8_MJ4CH2: now also MJ4.3 (ENC_CH2); no longer MJ1.3 (ENC_CH2)
- net PA9_MJ2CH1 renamed PA9_MJ4CH1
- net PA9_MJ4CH1: now also MJ4.4 (ENC_CH1); no longer MJ1.4 (ENC_CH1)
- net PB0_DR2AIN1 renamed PB0_DR1AIN1
- net PB0_DR1AIN1: now also DR1.21 (AIN1); no longer DR2.21 (AIN1)
- net PB10_DR2BIN2 renamed PB10_DR1BIN2
- net PB10_DR1BIN2: now also DR1.16 (BIN2); no longer DR2.16 (BIN2)
- net PB2_DR2BIN1 renamed PB2_DR1BIN1
- net PB2_DR1BIN1: now also DR1.17 (BIN1); no longer DR2.17 (BIN1)
- net PB3_DR1PWMA renamed PB3_DR2PWMA
- net PB3_DR2PWMA: now also DR2.23 (PWMA); no longer DR1.23 (PWMA)
- net PB4_DR1AIN1 renamed PB4_DR2AIN1
- net PB4_DR2AIN1: now also DR2.21 (AIN1); no longer DR1.21 (AIN1)
- net PB5_DR1AIN1 renamed PB5_DR2AIN1
- net PB5_DR2AIN1: now also DR2.22 (AIN2); no longer DR1.22 (AIN2)
- net PB6_MJ1CH1 renamed PB6_MJ2CH2
- net PB6_MJ2CH2: now also MJ2.3 (ENC_CH2); no longer MJ3.4 (ENC_CH1)
- net PB7_MJ1CH2 renamed PB7_MJ2CH1
- net PB7_MJ2CH1: now also MJ2.4 (ENC_CH1); no longer MJ3.3 (ENC_CH2)
- net PC14_DR1BIN1 renamed PC14_DR2BIN1
- net PC14_DR2BIN1: now also DR2.17 (BIN1); no longer DR1.17 (BIN1)
- net PC15_DR1BIN2 renamed PC15_DR2BIN2
- net PC15_DR2BIN2: now also DR2.16 (BIN2); no longer DR1.16 (BIN2)

Commit message: update
Connections:
- net PB5_DR2AIN1 renamed PB5_DR2AIN2
Changed lines of the file:
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@@
 		)
 	)
-	(label "PB5_DR2AIN1"
+	(label "PB5_DR2AIN2"
 		(at 22.86 82.55 0)
 		(effects
@@
 		)
 	)
-	(label "PB5_DR2AIN1"
+	(label "PB5_DR2AIN2"
 		(at 185.42 120.65 0)
 		(effects

Commit message: fix board design
Connections:
- net GND23: now also U1.23 (GND); no longer U1.24 (3V3)
Changed lines of the file:
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@@
+	)
+	(no_connect
+		(at 74.93 100.33)
 	)
 	(no_connect
@@
 	)
 	(no_connect
-		(at 74.93 102.87)
-	)
-	(no_connect
 		(at 148.59 110.49)
 	)
@@
 	(wire
 		(pts
-			(xy 74.93 100.33) (xy 78.74 100.33)
-		)
-		(stroke
-			(width 0)
-			(type default)
-		)
-	)
-	(wire
-		(pts
 			(xy 154.94 86.36) (xy 138.43 86.36)
 		)
@@
 		(pts
 			(xy 116.84 163.83) (xy 115.57 163.83)
+		)
+		(stroke
+			(width 0)
+			(type default)
+		)
+	)
+	(wire
+		(pts
+			(xy 74.93 102.87) (xy 78.74 102.87)
 		)
 		(stroke
@@
 	)
 	(label "GND23"
-		(at 78.74 100.33 0)
+		(at 78.74 102.87 0)
 		(effects
 			(font

Commit message: update borad 2
Parts:
- removed D1: GREEN_LED, LED_THT:LED_D3.0mm, symbol Device:LED
- removed S1, S2: INA226, LGDXRobot2:INA226, symbol Sensor_Energy:INA226
- added C1, C2, C3: 0.1uF, Capacitor_THT:C_Disc_D5.0mm_W2.5mm_P2.50mm, symbol Device:C
- added J2, J3, J4: PH2.0 2P, Connector_JST:JST_PH_B2B-PH-K_1x02_P2.00mm_Vertical, symbol Connector:Conn_01x02_Socket
- added R4: 68k, Resistor_THT:R_Axial_DIN0207_L6.3mm_D2.5mm_P7.62mm_Horizontal, symbol Device:R
- added R5, R6, R7: 10k, Resistor_THT:R_Axial_DIN0207_L6.3mm_D2.5mm_P7.62mm_Horizontal, symbol Device:R
- added S1: ~, LGDXRobot2:ICM20948, symbol LGDXRobot2_Library:ICM20948
- R2, R3: value 4k7 -> 68k
- renumbered D2 to D1
Connections:
- net 5V99: no longer R2.1, R3.1
- net GND47: now also S1.2 (GND)
- net PC13_DR2BIN2: now reaches U1.2 (PC13)
- net PC13_DR2BIN2: now also DR2.16 (BIN2)
- net PB12_DR1BIN1: now reaches U1.25 (PB12)
- net PB12_DR1BIN1: now also DR1.17 (BIN1)
- net PB13_DR1BIN2: now reaches U1.26 (PB13)
- net PB13_DR1BIN2: now also DR1.16 (BIN2)
- net PB14_ADO: now reaches U1.27 (PB14)
- net PB14_ADO: now also S1.6 (ADO)
- net 3V348: now reaches U1.48 (3V3)
- net 3V348: now also S1.1 (VCC)
- net PA0_MJ3CH2 renamed PA0_MJ3CH1
- net PA0_MJ3CH1: now also MJ3.4 (ENC_CH1); no longer MJ3.3 (ENC_CH2)
- net PA10_D2 renamed PA10_NCS
- net PA10_NCS: now also S1.5 (NCS); no longer D1.2 (A)
- net PA15_RS1 renamed PA15_DR2BIN1
- net PA15_DR2BIN1: now also DR2.17 (BIN1); no longer RS1.3 (INPUT)
- net PA1_MJ3CH1 renamed PA1_MJ3CH2
- net PA1_MJ3CH2: now also MJ3.3 (ENC_CH2); no longer MJ3.4 (ENC_CH1)
- net PA4_DR1AIN2 renamed PA4_ESTOP
- net PA4_ESTOP: now also C3.1, R4.2, R7.1; no longer DR1.22 (AIN2)
- net PB0_DR1AIN1 renamed PB0_BT2
- net PB0_BT2: now also R3.2, C2.1, R6.1; no longer DR1.21 (AIN1)
- net PB10_DR1BIN2 renamed PB10_SCLK
- net PB10_SCLK: now also S1.3 (SCLK); no longer DR1.16 (BIN2)
- net PB15_D1 renamed PB15_SDA
- net PB15_SDA: now also S1.4 (SDI)
- net PB1_DRxSTBY renamed PB2_DRxSTBY
- net PB2_DRxSTBY: now also U1.20 (PB2); no longer U1.19 (PB1)
- removed net PB2_DR1BIN1: DR1.17 (BIN1), U1.20 (PB2)
- net PB8_SCL renamed PB8_D1
- net PB8_D1: now also D1.2 (A); no longer R3.2
- net PB9_SDA renamed PB1_BT1
- net PB1_BT1: now also U1.19 (PB1), C1.1, R5.1; no longer U1.46 (PB9)
- net PC14_DR2BIN1 renamed PC14_DR1AIN2
- net PC14_DR1AIN2: now also DR1.22 (AIN2); no longer DR2.17 (BIN1)
- net PC15_DR2BIN2 renamed PC15_DR1AIN1
- net PC15_DR1AIN1: now also DR1.21 (AIN1); no longer DR2.16 (BIN2)
- new net: J3.2 (Pin_2), R3.1
- new net: C3.2, J4.1 (Pin_1), R7.2
- new net: J4.2 (Pin_2), R4.1
- new net: C1.2, J2.1 (Pin_1), R5.2
- new net: C2.2, J3.1 (Pin_1), R6.2
- new net: J2.2 (Pin_2), R2.1
- new net PB9_RS1: RS1.3 (INPUT), U1.46 (PB9)
- no-connect marks 26 -> 17
Other:
- note added: "E-STOP Indicator / Relay"
- note added: "IMU"
- note removed: "Software E-STOP & Indicator"
- title: LGDXRobot2 Board -> LGDXRobot2 Board V2
- moved on the sheet: D1, R1, RS1
