File: Board/Board.kicad_sch (KiCad schematic)
At the start: 24 parts, among them J1 XT30 Female, J2 PH2.0 2P, J3 PH2.0 2P, J4 PH2.0 2P, U1 BlackPill

Commit message: board v2 pcb
Connections:
- net GND47: now also DR1.18 (GND), DR2.18 (GND), MJ1.5 (ENC_GND), MJ2.5 (ENC_GND), MJ3.5 (ENC_GND), MJ4.5 (ENC_GND)
- removed net GND23: DR1.18 (GND), DR2.18 (GND), MJ1.5 (ENC_GND), MJ2.5 (ENC_GND), MJ3.5 (ENC_GND), MJ4.5 (ENC_GND), U1.23 (GND)
- net PA3_DR1PWMA renamed PA3_DR1PWMB
- net PA3_DR1PWMB: now also DR1.15 (PWMB); no longer DR1.23 (PWMA)
- net PA5_DR1PWMB renamed PA5_DR1PWMA
- net PA5_DR1PWMA: now also DR1.23 (PWMA); no longer DR1.15 (PWMB)
- net PB12_DR1BIN1 renamed PB12_DR1BIN2
- net PB12_DR1BIN2: now also DR1.16 (BIN2); no longer DR1.17 (BIN1)
- net PB13_DR1BIN2 renamed PB13_DR1BIN1
- net PB13_DR1BIN1: now also DR1.17 (BIN1); no longer DR1.16 (BIN2)
- no-connect marks 17 -> 18
Changed lines of the file:
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@@
+	)
+	(no_connect
+		(at 74.93 102.87)
 	)
 	(no_connect
@@
 		(pts
 			(xy 123.19 41.91) (xy 123.19 48.26)
-		)
-		(stroke
-			(width 0)
-			(type default)
-		)
-	)
-	(wire
-		(pts
-			(xy 74.93 102.87) (xy 78.74 102.87)
 		)
 		(stroke
@@
 		)
 	)
-	(label "PB12_DR1BIN1"
+	(label "PB12_DR1BIN2"
 		(at 22.86 97.79 0)
 		(effects
@@
 		)
 	)
-	(label "GND23"
-		(at 78.74 102.87 0)
-		(effects
-			(font
-				(size 1.27 1.27)
-			)
-			(justify left bottom)
-		)
-	)
 	(label "PA10_NCS"
 		(at 78.74 67.31 0)
@@
 		)
 	)
-	(label "PB13_DR1BIN2"
+	(label "PB12_DR1BIN2"
 		(at 185.42 64.77 0)
 		(effects
@@
 		)
 	)
-	(label "PA3_DR1PWMA"
+	(label "PA3_DR1PWMB"
 		(at 78.74 49.53 0)
 		(effects
@@
 		)
 	)
-	(label "PA5_DR1PWMB"
+	(label "PA3_DR1PWMB"
 		(at 185.42 52.07 0)
 		(effects
@@
 		)
 	)
-	(label "PB13_DR1BIN2"
+	(label "PB13_DR1BIN1"
 		(at 22.86 100.33 0)
 		(effects
@@
 		)
 	)
-	(label "PA3_DR1PWMA"
+	(label "PA5_DR1PWMA"
 		(at 185.42 49.53 0)
 		(effects
@@
 		)
 	)
-	(label "PA5_DR1PWMB"
+	(label "PA5_DR1PWMA"
 		(at 78.74 54.61 0)
 		(effects
@@
 		)
 	)
-	(label "GND23"
+	(label "GND47"
 		(at 256.54 143.51 0)
 		(effects
@@
 		)
 	)
-	(label "PB12_DR1BIN1"
+	(label "PB13_DR1BIN1"
 		(at 185.42 62.23 0)
 		(effects
